File: _autosave-ai03-pcb-guide-TPS.kicad_pcb (KiCad board)
At the start: 2 copper layers, 73.8 x 38.1 mm, 24 parts, among them SW1 SW_Push, U1 ATmega32U4-AU, Y1 16MHz

Commit message: Update _autosave-ai03-pcb-guide-TPS.kicad_pcb
Connections:
- U1 pad 27: Net-(U1-Pad27) -> ROW0
- U1 pad 28: Net-(U1-Pad28) -> COL1
- U1 pad 29: Net-(U1-Pad29) -> COL0
- U1 pad 30: Net-(U1-Pad30) -> ROW1
Routing:
- net COL1: track 0.00 -> 53.1 mm
- net ROW1: track 0.00 -> 49.9 mm
- net ROW0: track 0.00 -> 47.6 mm
- net COL0: track 0.00 -> 33.7 mm
- net Net-(D4-Pad2): track 0.00 -> 6.62 mm
- net Net-(D3-Pad2): track 0.00 -> 6.62 mm
- net Net-(D2-Pad2): track 0.00 -> 6.62 mm
- net Net-(D1-Pad2): track 0.00 -> 6.62 mm
